File: FAL6567/trunk/sch/FAL6567.sch (EAGLE design)
At the start: 6 parts, among them IC1 74LS245DW, IC2 74LS245DW, IC3 74LS245DW, IC4 74LS245DW

Commit message: FAL6567 Update
Parts:
- added D1, D2: 1N4004, diode:1N4004
- added IC5: 74LS06D, FT74xx:74LS06D
- added R1, R5: 2k, resistor:R-US_0207/10
- added R10, R3, R7: 510, resistor:R-US_0207/10
- added R13, R14: 100, resistor:R-US_0207/10
- added R2, R6, R9: 1k, resistor:R-US_0207/10
- added X1: (no value), con-subd:F15HDV
Connections:
- removed net N$11: IC2A.B3
- removed net N$14: IC2A.B6
- removed net N$16: IC2A.B8
- removed net N$9: IC2A.B1
- new net +5V: D2.A, U$1.VCC
- new net A0: IC1A.B8, U$2.PIO26
- new net A1: IC1A.B7, U$2.PIO27
- new net A10: IC4A.B1, U$2.PIO16
- new net A11: IC4A.B4, U$2.PIO19
- new net A2: IC1A.B6, U$2.PIO28
- new net A3: IC1A.B5, U$2.PIO29
- new net A4: IC1A.B4, U$2.PIO30
- new net A5: IC1A.B3, U$2.PIO31
- new net A6: IC1A.B2, U$2.PIO32
- new net A7: IC1A.B1, U$2.PIO33
- new net A8: IC4A.B3, U$2.PIO18
- new net A9: IC4A.B2, U$2.PIO17
- new net BA: IC4A.B6, U$2.PIO21
- new net BLUE0: R9.1, U$2.PIO40
- new net BLUE1: R10.1, U$2.PIO39
- new net CAS: IC4A.B8, U$2.PIO23
- new net CSB: IC3A.B5, U$2.PIO13
- new net D0: IC2A.B8, U$2.PIO8
- new net D1: IC2A.B7, U$2.PIO7
- new net D10: IC3A.B3, U$2.PIO11
- new net D11: IC3A.B4, U$2.PIO12
- new net D2: IC2A.B6, U$2.PIO6
- new net D3: IC2A.B5, U$2.PIO5
- new net D4: IC2A.B4, U$2.PIO4
- new net D5: IC2A.B3, U$2.PIO3
- new net D6: IC2A.B2, U$2.PIO2
- new net D7: IC2A.B1, U$2.PIO1
- new net D8: IC3A.B1, U$2.PIO9
- new net D9: IC3A.B2, U$2.PIO10
- new net GREEN0: R5.1, U$2.PIO44
- new net GREEN1: R6.1, U$2.PIO43
- new net GREEN2: R7.1, U$2.PIO42
- new net HSYNC: R14.1, U$2.PIO36
- new net IRQ: IC5A.I, U$2.PIO37
- new net LPB: IC3A.B7, U$2.PIO15
- new net N$1: IC5A.O, U$1.IRQB
- new net N$2: U$2.GND
- new net N$3: D1.C, U$2.VU
- new net N$4: IC5B.O
- new net N$6: D1.A, D2.C
- new net N$7: R1.2, R2.2, R3.2, X1.1
- new net PHI02: IC3A.A8, U$2.PIO45
- new net RAS: IC4A.B7, U$2.PIO22
- new net RED0: R1.1, U$2.PIO48
- new net RED1: R2.1, U$2.PIO47
- new net RED2: R3.1, U$2.PIO46
- new net RESET: IC5B.I, U$2.PIO34
- new net RWB: IC3A.B6, U$2.PIO14
- new net VPHI02: IC3A.B8, U$1.PHI0
- new net VSYNC: R13.1, U$2.PIO35
- net AEC: now also IC4A.B5, U$2.PIO20
- net DEN: now also U$2.PIO41
- net DIR: now also U$2.PIO38
- net GND: now also U$1.GND, X1.10, X1.5, X1.6, X1.7, X1.8, X1.9
- net N$10: now also R10.2, R9.2, X1.3; no longer IC2A.B2
- net N$12: now also R14.2, X1.13; no longer IC2A.B4
- net N$13: now also R13.2, X1.14; no longer IC2A.B5
- net N$15: now also R5.2, R6.2, R7.2, X1.2; no longer IC2A.B7
- net VA0: now also IC1A.A8; no longer IC1A.A1
- net VA1: now also IC1A.A7; no longer IC1A.A2
- net VA10: now also IC4A.A1; no longer IC4A.A3
- net VA2: now also IC1A.A6; no longer IC1A.A3
- net VA3: now also IC1A.A5; no longer IC1A.A4
- net VA4: now also IC1A.A4; no longer IC1A.A5
- net VA5: now also IC1A.A3; no longer IC1A.A6
- net VA6: now also IC1A.A2; no longer IC1A.A7
- net VA7: now also IC1A.A1; no longer IC1A.A8
- net VA8: now also IC4A.A3; no longer IC4A.A1
- net VD0: now also IC2A.A8; no longer IC2A.A1
- net VD1: now also IC2A.A7; no longer IC2A.A2
- net VD2: now also IC2A.A6; no longer IC2A.A3
- net VD3: no longer IC2A.A4
- net VD4: now also IC2A.A4
- net VD5: now also IC2A.A3; no longer IC2A.A6
- net VD6: now also IC2A.A2; no longer IC2A.A7
- net VD7: now also IC2A.A1; no longer IC2A.A8

Commit message: FAL6567 - Latest Files
Parts:
- removed D1: 1N4004, diode:1N4004
- removed R7: 510, resistor:R-US_0207/10
- added C1, C2, C3: (no value), resistor:C-EU050-024X044
- added C4: 0.1, resistor:C-EU050-024X044
- added C5, C6: 10u, resistor:C-USC1206
- added IC6: REG1117F, burr-brown:REG1117F
- added JP1: (no value), jumper:JP1E
- added JP2: (no value), jumper:JP3Q
- R1, R5: value 2k -> 1k; device resistor:R-US_0207/10 -> resistor:R-US_0204/7
- R10, R13, R14, R9: device resistor:R-US_0207/10 -> resistor:R-US_0204/7
- R2, R6: value 1k -> 510; device resistor:R-US_0207/10 -> resistor:R-US_0204/7
- R3: value 510 -> 4.7k; device resistor:R-US_0207/10 -> resistor:R-US_0204/7
Connections:
- removed net +3V3: IC3A.DIR
- removed net GREEN2: R7.1, U$2.PIO42
- removed net N$2: U$2.GND
- removed net N$3: D1.C, U$2.VU
- removed net N$6: D1.A, D2.C
- removed net RED2: R3.1, U$2.PIO46
- new net MD0: JP2.4, U$2.PIO15
- new net MD1: JP2.3, U$2.PIO16
- new net N$8: IC5B.O, JP1.1, JP1.2
- new net VCC: C1.1, C2.1, C3.1, C4.1, C6.1, IC3A.DIR, IC6.VOUT, JP2.1, JP2.2, R3.2
- net +5V: now also C5.1, IC6.VIN
- net A10: now also U$2.PIO46; no longer U$2.PIO16
- net GND: now also C1.2, C2.2, C3.2, C4.2, C5.2, C6.2, IC5C.I, IC5D.I, IC5E.I, IC5F.I, IC6.GND, JP2.5, JP2.6, U$2.GND
- net LPB: now also U$2.PIO42; no longer U$2.PIO15
- net N$15: no longer R7.2
- net N$4: now also D2.C, U$2.VU; no longer IC5B.O
- net N$7: no longer R3.2
- net RESET: now also R3.1
- net VA1: now also U$1.A1/A9
- net VD3: now also IC2A.A5
Other:
- moved on the sheet: R3
