File: FAL6567/trunk/sch/FAL65816_6567a.sch (EAGLE design)
At the start: 34 parts, among them IC1 74LVC04D, IC10 74LVC245DW, IC12 74LVC00D, IC13 74LVC138D, IC2 74LVC245DW, IC4 74LVC573, IC5 74LVC573, IC7 74LVC573, Q1 2N2222, U1 65C22

Commit message: FAL65816 - update
Parts:
- removed U1: 65C22, 65xxx:G65SC22P
- added JP3: (no value), pinhead:PINHD-1X4/90
- JP1: device pinhead:PINHD-2X25 -> pinhead:PINHD-2X25/90
Connections:
- removed net C6522N: IC13A.Y2, U1.CS2B
- removed net PA0: IC5A.7D, U1.PA0
- removed net PA1: IC5A.8D, U1.PA1
- removed net PA2: IC7A.1D, U1.PA2
- removed net PA3: IC7A.2D, U1.PA3
- removed net PA4: IC7A.3D, U1.PA4
- removed net PA5: IC7A.4D, U1.PA5
- removed net PA6: IC7A.5D, U1.PA6
- removed net PA7: IC7A.6D, U1.PA7
- new net CSAH: IC1B.O, IC7A.C
- new net CSAHN: IC13A.Y2, IC1B.I
- net +12V: now also JP3.4
- net A11: no longer U1.CS1
- net A14: now also IC7A.1Q; no longer IC5A.7Q
- net A15: now also IC7A.2Q; no longer IC5A.8Q
- net A16: now also IC7A.3Q; no longer IC7A.1Q
- net A17: now also IC7A.4Q; no longer IC7A.2Q
- net A18: now also IC7A.5Q; no longer IC7A.3Q
- net A19: now also IC7A.6Q; no longer IC7A.4Q
- net A20: now also IC7A.7Q; no longer IC7A.5Q
- net A21: now also IC7A.8Q; no longer IC7A.6Q
- net A22: now also IC5A.7Q; no longer IC7A.7Q
- net A23: now also IC5A.8Q; no longer IC7A.8Q
- net D0: now also IC7A.1D; no longer U1.D0
- net D1: now also IC7A.2D; no longer U1.D1
- net D2: now also IC7A.3D; no longer U1.D2
- net D3: now also IC7A.4D; no longer U1.D3
- net D4: now also IC7A.5D; no longer U1.D4
- net D5: now also IC7A.6D; no longer U1.D5
- net D6: now also IC7A.7D; no longer U1.D6
- net D7: now also IC7A.8D; no longer U1.D7
- net GND: now also IC5A.7D, IC5A.8D, JP3.2, JP3.3; no longer IC1B.I, IC7A.7D, IC7A.8D, U1.VSS
- net IRQN: no longer U1.IRQB
- net PH2: no longer U1.PH2
- net PU1: no longer IC7A.C
- net RESN: no longer U1.RESB
- net RWB: no longer U1.R/WB
- net VA0: no longer U1.RS0
- net VA1: no longer U1.RS1
- net VA2: no longer U1.RS2
- net VA3: no longer U1.RS3
- net VCC: now also JP3.1; no longer U1.VDD
Other:
- moved on the sheet: C1, C2, C3, C4, IC1B, JP2, L1, Q1, R1, R2, R3, R4
