File: FAL6567/trunk/sch/FAL65816_Audio.sch (EAGLE design)
At the start: 31 parts, among them IC1 74LS688DW, IC2 74LS00D, Q1 2N2222, U2 65C22

Commit message: FAL65816 - update
Parts:
- added C12, C13, C15, C16: 0.1, resistor:C-US050-024X044
- added C17: 10, resistor:C-US050-024X044
- added JP10: 5V Serial Port, pinhead:PINHD-1X6/90
- added JP9: POWER, pinhead:PINHD-1X4/90
- added U$2: OSC, FT74xx:OSC
- added U1: 65C51, 65xxx:G65SC51P
- IC2: value 74LS00D -> 74LS138D; device FT74xx:74LS00D -> FT74xx:74LS138D
- JP1: device pinhead:PINHD-2X25 -> pinhead:PINHD-2X25/90
- JP2: value (none) -> AUDIO OUT
- JP3: value (none) -> EXT IN
- JP4: value (none) -> POTX
- JP5: value (none) -> POTY
- JP6: value (none) -> KEYBOARD PORT
- JP8: device pinhead:PINHD-1X6 -> pinhead:PINHD-1X6/90
Connections:
- removed net N$10: JP3.2, JP4.2, JP5.2
- removed net N$14: IC2B.I1, IC2C.O
- removed net N$15: IC1A.Q4, IC1A.Q6, R1.1
- new net CS6522N: IC2A.Y1, U2.CS2B
- new net CS6551N: IC2A.Y2, U1.CS1B
- new net N$20: JP10.4, U1.TXD
- new net N$21: JP10.5, U1.RXD
- new net N$22: JP10.6, U1.RTS
- new net N$28: U$2.OUT, U1.XTL1
- new net PU1: IC1A.Q7, IC2A.G1, R1.1, U1.CS0, U2.CS1
- net +12V: now also JP9.4
- net A0: now also U1.RS0
- net A1: now also U1.RS1
- net A5: now also IC2A.A
- net A6: now also IC2A.B
- net A7: now also IC2A.C; no longer IC2A.I0, IC2A.I1, U2.CS1
- net CS6581N: now also IC2A.Y0; no longer IC2B.O
- net CSN: now also IC2A.G2A; no longer IC2C.I0, IC2C.I1, U2.CS2B
- net D0: now also U1.D0
- net D1: now also U1.D1
- net D2: now also U1.D2
- net D3: now also U1.D3
- net D4: now also U1.D4
- net D5: now also U1.D5
- net D6: now also U1.D6
- net D7: now also U1.D7
- net GND: now also C12.2, C13.2, C15.2, C16.2, C17.2, IC1A.Q4, IC1A.Q6, IC2A.G2B, JP10.1, JP3.2, JP4.2, JP5.2, JP9.2, JP9.3, U$2.GND, U1.DCD, U1.DSR, U1.VSS; no longer IC1A.Q7, IC2D.I0, IC2D.I1
- net IRQN: now also U1.IRQB
- net N$17: now also JP10.2, U1.CTS; no longer IC2A.O, IC2B.I0
- net PH2: now also U1.PH2
- net RESN: now also U1.RESB
- net RW: now also U1.R/WB
- net VCC: now also C12.1, C13.1, C15.1, C16.1, C17.1, JP10.3, JP9.1, U$2.VCC, U1.VDD
Other:
- note added: "SID = $FD80xx"
- note added: "nc"
- note removed: "SID = $FD50xx"
