File: FAL6567/trunk/sch/FAL65816_ram.brd (EAGLE design)
At the start: 100 x 80 mm, 18 parts, among them IC1 74LS688DW, IC11 74259D, IC12 74LS00D, IC2 27C512, IC4 74LS688DW, IC6 74LS138D

Commit message: FAL65816 - update
Parts:
- added JP3: POWER, pinhead:1X04/90
- IC2: value 27C512 -> 27C256
- JP1: value (none) -> RAM BUS Conn
- JP2: value (none) -> System Bus Conn; device pinhead:2X25 -> pinhead:2X25/90
- R1: value (none) -> 3k3
- moved C5 12.0 mm to (73.7, 38.1)
- moved JP1 7.73 mm to (25.4, 41.9)
- moved C3 7.62 mm to (47.0, 40.6)
- moved IC6 7.62 mm to (47.0, 48.3)
- moved C1 6.35 mm to (45.7, 59.7)
- moved IC11 6.35 mm to (45.7, 67.3)
- moved LED1 5.08 mm to (96.5, 35.6), turned to 270 degrees
- moved JP2 4.02 mm to (50.8, 0.00), turned to 180 degrees
- moved C4 3.81 mm to (63.5, 41.9)
- moved IC12 3.81 mm to (63.5, 48.3)
- moved IC2 3.81 mm to (85.1, 58.4)
- moved R2 3.81 mm to (83.8, 33.0)
- moved C6 2.54 mm to (58.4, 20.3)
- moved IC4 2.54 mm to (67.3, 20.3)
- moved C2 1.27 mm to (63.5, 58.4)
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Connections:
- new net +12V: JP3.4
- new net N$4: IC12.6, IC4.2
- net A15: now also IC12.4; no longer IC2.1
- net A16: now also IC12.5; no longer IC4.2
- net GND: now also JP3.2, JP3.3; no longer IC12.4, IC12.5
- net PU1: now also IC2.1
- net VCC: now also JP3.1
Routing:
- net A20: track 69.3 -> 304.3 mm
- net A21: track 82.4 -> 235.2 mm, vias 4 -> 8
- net GND: track 278.4 -> 411.2 mm, vias 10 -> 9
- net D7: track 53.1 -> 183.9 mm, vias 3 -> 8
- net D3: track 215.5 -> 123.9 mm, vias 5 -> 8
- net D6: track 113.0 -> 203.4 mm, vias 5 -> 7
- net A0: track 140.8 -> 217.6 mm, vias 4 -> 11
- net PH2: track 144.8 -> 71.2 mm, vias 4 -> 5
- net A1: track 146.7 -> 214.8 mm, vias 10 -> 5
- net A4: track 166.6 -> 104.5 mm, vias 5 -> 3
- net A19: track 80.5 -> 140.9 mm, vias 1 -> 3
- net A10: track 173.1 -> 230.1 mm, vias 5 -> 4
- net A11: track 168.8 -> 222.3 mm, vias 8 -> 7
- net A22: track 24.4 -> 74.5 mm, vias 0 -> 3
- net A5: track 163.0 -> 210.8 mm
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