File: FAL6567/trunk/sch/FAL65816_ram.sch (EAGLE design)
At the start: 18 parts, among them IC1 74LS688DW, IC11 74259D, IC12 74LS00D, IC2 27C512, IC4 74LS688DW, IC6 74LS138D

Commit message: FAL65816 - update
Parts:
- added JP3: POWER, pinhead:PINHD-1X4/90
- IC2: value 27C512 -> 27C256; device memory:27512 -> memory:27256
- JP1: value (none) -> RAM BUS Conn
- JP2: value (none) -> System Bus Conn; device pinhead:PINHD-2X25 -> pinhead:PINHD-2X25/90
- R1: value (none) -> 3k3
Connections:
- new net +12V: JP3.4
- new net N$4: IC12B.O, IC4A.P0
- net A15: now also IC12B.I0; no longer IC2A.A15
- net A16: now also IC12B.I1; no longer IC4A.P0
- net GND: now also JP3.2, JP3.3; no longer IC12B.I0, IC12B.I1
- net PU1: now also IC2A.VPP
- net VCC: now also JP3.1
Other:
- moved on the sheet: IC12A, IC12B, IC12C, IC12D
