File: ISA/ISA_FPGA/ISA_FPGA.sch (KiCad schematic (older format))
At the start: 44 parts, among them J1 Bus_ISA_16bit, J2 DE15, P1 CONN_5X2, P2 14.31818MHz, U1 74LVC245, U2 74LVC245, U3 74LVC245, U4 74LVC245, U5 74LVC245, U6 74LVC245, U7 CONN_30X2, U8 CONN_30X2, U9 74LVC06, X1 MINI_DIN_6, X2 MINI_DIN_6

Commit message: ISA - FPGA board
Parts:
- added C?: 0.1, ~, symbol FPGA-Board-rescue:C
- added C?: 10uF, ~, symbol FPGA-Board-rescue:CAPAPOL
- added D? (x27): ZPDxx, Diode_THT:D_DO-35_SOD27_P10.16mm_Horizontal, symbol Diode:ZPDxx
- added D? (x4): LED, Diode_THT:D_DO-35_SOD27_P10.16mm_Horizontal, symbol VGA~V11-cache:LED
- added P?: CONN_6, ~, symbol FPGA-Board-rescue:CONN_6
- added P?: CONN_2X2, ~, symbol FPGA-Board-rescue:CONN_2X2
- added P? (x2): CONN_7, ~, symbol FPGA-Board-rescue:CONN_7
- added P?: CONN_2, ~, symbol FPGA-Board-rescue:CONN_2
- added P?: CONN_5X2, symbol VGA~V11-cache:CONN_5X2
- added R?: 10K, ~, symbol FPGA-Board-rescue:R
- added R? (x24): 200, symbol VGA_V11-cache:R
- added R? (x7): 100, symbol VGA_V11-cache:R
- added RR?: 10k, Resistor_THT:R_Array_SIP10, symbol VGA~V11-cache:RR9
- added U?: LM3940, ~, symbol FPGA-Board-rescue:7805
- added U? (x3): CONN_6x2, Connector_PinHeader_2.54mm:PinHeader_2x06_P2.54mm_Horizontal, symbol VGA_V11-cache:CONN_6x2
- added U?: CONN_6x2, symbol VGA~V11-cache:CONN_6x2
Connections:
- net labels added: 328_RESET*, ANA0, ANA1, ANA2, CFG0, CFG1, CFG2, CFG3, CFG4, CFG5, FRX, FTX, LED0, LED1, LED2, LED3, PMODA0, PMODA1, PMODA2, PMODA3, PMODA4, PMODA5, PMODA6, PMODA7, PMODB0, PMODB1, PMODB2, PMODB3, PMODB4, PMODB5, PMODB6, PMODB7, PMODC0, PMODC1, PMODC2, PMODC3, PMODC4, PMODC5, PMODC6, PMODC7
- wire segments 377 -> 723
- no-connect marks 0 -> 13
Other:
- note added: "Analog"
- note added: "Normally Open\n(USB supplies 5V)"
- note added: "SparkFun\nFT231x\nSerial->USB"
- note added: "VREF"
- moved on the sheet: C1, C2, C3, C4, C5, C6, C7

Commit message: ISA - update
cad files for ISA video / cpu boards
Parts:
- removed D? (x8): ZPDxx, Diode_THT:D_DO-35_SOD27_P10.16mm_Horizontal, symbol Diode:ZPDxx
- removed P2: 14.31818MHz, Package_DIP:DIP-14_W7.62mm_Socket, symbol VGA~V11-cache:DIL14
- removed R22: 2k2, Resistor_THT:R_Axial_DIN0207_L6.3mm_D2.5mm_P7.62mm_Horizontal, symbol VGA~V11-cache:R
- removed R? (x12): 200, symbol VGA_V11-cache:R
- removed U7, U8: CONN_30X2, Connector_PinSocket_2.54mm:PinSocket_2x30_P2.54mm_Vertical, symbol VGA~V11-cache:CONN_30X2
- removed unit 1 of U9
- removed unit 2 of U9
- removed U?: CONN_6x2, Connector_PinHeader_2.54mm:PinHeader_2x06_P2.54mm_Horizontal, symbol VGA_V11-cache:CONN_6x2
- added C10, C11: 0.1, Capacitor_THT:C_Disc_D3.0mm_W1.6mm_P2.50mm, symbol VGA~V11-cache:CP1
- added D1: LED, Diode_THT:D_DO-35_SOD27_P10.16mm_Horizontal, symbol VGA~V11-cache:LED
- added JP1, JP2: Jumper, Connector_PinHeader_2.54mm:PinHeader_1x02_P2.54mm_Vertical, symbol Device:Jumper
- added R28: 100, Resistor_THT:R_Axial_DIN0207_L6.3mm_D2.5mm_P7.62mm_Horizontal, symbol VGA_V11-cache:R
- added U10: 74LVC245, Package_SO:SOIC-20W_7.5x12.8mm_P1.27mm, symbol 74xx:74LS245
- added U15: 74LVC138, Package_SO:SOIC-16W_7.5x10.3mm_P1.27mm, symbol 74xx:74LS138
- added U17: 74LVC574, Package_SO:SOIC-20W_7.5x12.8mm_P1.27mm, symbol 74xx:74LS574
- added U7, U8: CONN_32X2, Connector_PinSocket_2.54mm:PinSocket_2x32_P2.54mm_Vertical, symbol VGA~V11-cache:CONN_32X2
- added unit 5 of U9
- added unit 7 of U9
- C8: renamed from C?; footprint ~ -> Capacitor_THT:C_Disc_D3.0mm_W1.6mm_P2.50mm
- C9: renamed from C?; footprint ~ -> Capacitor_THT:CP_Radial_D7.5mm_P2.50mm
- P3: renamed from P?; footprint (none) -> Connector_PinHeader_2.54mm:PinHeader_2x05_P2.54mm_Vertical
- P4, P7: renamed from P?; footprint ~ -> Connector_PinSocket_2.54mm:PinSocket_1x07_P2.54mm_Vertical
- P5: renamed from P?; footprint ~ -> Connector_PinSocket_2.54mm:PinSocket_1x06_P2.54mm_Vertical
- P6: renamed from P?; footprint ~ -> Connector_PinHeader_2.54mm:PinHeader_2x02_P2.54mm_Vertical
- P8: renamed from P?; footprint ~ -> Connector_PinHeader_2.54mm:PinHeader_1x02_P2.54mm_Vertical
- R23, R24, R25, R26, R31, R32, R33, R34, R35, R36, R37, R38, R39, R40, R41, R51, R52, R53, R54: renamed from R?; footprint (none) -> Resistor_THT:R_Axial_DIN0207_L6.3mm_D2.5mm_P7.62mm_Horizontal
- R50: renamed from R?; footprint ~ -> Resistor_THT:R_Axial_DIN0207_L6.3mm_D2.5mm_P7.62mm_Horizontal
- U11, U12: renamed from U?; footprint Connector_PinHeader_2.54mm:PinHeader_2x06_P2.54mm_Horizontal -> Connector_PinSocket_2.54mm:PinSocket_2x06_P2.54mm_Horizontal
- U13: renamed from U?; footprint (none) -> Connector_PinHeader_2.54mm:PinHeader_2x06_P2.54mm_Vertical
- U14: renamed from U?; footprint ~ -> Package_TO_SOT_THT:LMxx
- gave numbers to parts that had none: 24
Connections:
- net labels added: 14M318Hz, 8M18Hz, 8MH18Hz, A0, F14M318Hz, F8M18Hz, FMEMCS16, FMRQ0, FMRQ1, FMRQ2, FMRQ3, FMRQ5, FMRQ6, FMRQ7, FSBHE, FWR*, LED4, MAK0*, MAK1*, MAK2*, MAK3*, MAK5*, MAK6*, MAK7*, MEMCS16*, MOE*, MRQ0, MRQ1, MRQ2, MRQ3, MRQ5, MRQ6, MRQ7, MS0, MS1, MS2, RD*, RESET, SBHE
- net labels removed: CFG0, CFG1, CFG5, CYC, FSEL0, FSEL1, FWR, OSC, PMODB4, PMODB5, PMODB6, PMODB7, PMODC0, PMODC1, PMODC2, PMODC3, PMODC4, PMODC5, PMODC6, PMODC7, SEL0, SEL1
- wire segments 723 -> 697
Other:
- moved on the sheet: C1, C2, C3, C4, C5, C6, C7, C9, U14

Commit message: Petajon - update
Parts:
- removed D11, D12, D16, D18, D19, D2, D21, D22, D24, D25, D27, D3, D5, D6, D8, D9: ZPDxx, Diode_THT:D_DO-35_SOD27_P10.16mm_Horizontal, symbol Diode:ZPDxx
- removed R19: 2k2, Resistor_THT:R_Axial_DIN0207_L6.3mm_D2.5mm_P7.62mm_Horizontal, symbol VGA~V11-cache:R
- removed R25, R26, R31, R32, R33, R34, R38, R39, R40, R41: 200, Resistor_THT:R_Axial_DIN0207_L6.3mm_D2.5mm_P7.62mm_Horizontal, symbol VGA_V11-cache:R
- removed U11, U12: CONN_6x2, Connector_PinSocket_2.54mm:PinSocket_2x06_P2.54mm_Horizontal, symbol VGA_V11-cache:CONN_6x2
- removed U4: 74LVC245, Package_SO:SOIC-20W_7.5x12.8mm_P1.27mm, symbol 74xx:74LS245
- added C12: 0.047u, Capacitor_THT:C_Disc_D3.8mm_W2.6mm_P2.50mm, symbol Device:CP1
- added C13: 10u, Capacitor_THT:CP_Radial_D5.0mm_P2.50mm, symbol Device:CP1
- added C14: 100u, Capacitor_THT:CP_Radial_D8.0mm_P3.80mm, symbol Device:CP1
- added C15: 0.047u, Capacitor_THT:C_Disc_D5.0mm_W2.5mm_P5.00mm, symbol Device:CP1
- added C16: 220u, Capacitor_THT:CP_Radial_D8.0mm_P3.80mm, symbol Device:CP1
- added C17, C18, C19, C20, C21, C22, C23, C24: 0.1, Capacitor_THT:C_Disc_D3.0mm_W1.6mm_P2.50mm, symbol VGA~V11-cache:CP1
- added J3: AudioJack2, Connector_Audio:Jack_3.5mm_CUI_SJ1-3533NG_Horizontal, symbol Connector:AudioJack2
- added P2: CONN_2, Connector_PinHeader_2.54mm:PinHeader_1x02_P2.54mm_Vertical, symbol FPGA-Board-rescue:CONN_2
- added R19, R22: 10k, Resistor_THT:R_Axial_DIN0207_L6.3mm_D2.5mm_P7.62mm_Horizontal, symbol VGA_V11-cache:R
- added R27, R29: 5k1, Resistor_THT:R_Axial_DIN0207_L6.3mm_D2.5mm_P7.62mm_Horizontal, symbol VGA_V11-cache:R
- added R30: 10, Resistor_THT:R_Axial_DIN0207_L6.3mm_D2.5mm_P7.62mm_Horizontal, symbol VGA_V11-cache:R
- added R? (x8): 200, Resistor_THT:R_Axial_DIN0207_L6.3mm_D2.5mm_P7.62mm_Horizontal, symbol VGA_V11-cache:R
- added U11: 74LVC244, Package_SO:SOIC-20W_7.5x12.8mm_P1.27mm, symbol 74xx:74LS244
- added U12, U18, U4: 74LVC257, Package_SO:SOIC-16W_7.5x10.3mm_P1.27mm, symbol 74xx:74LS257
- added U16: LM386, Package_DIP:DIP-8_W7.62mm_Socket, symbol Amplifier_Audio:LM386
- added U19: CONN_20X2, Connector_PinHeader_2.54mm:PinHeader_2x20_P2.54mm_Horizontal, symbol VGA~V11-cache:CONN_20X2
- added U20: 74LVC573, Package_SO:SOIC-20W_7.5x12.8mm_P1.27mm, symbol 74xx:74LS573
- added U21, U22: 74LVC245, Package_SO:SOIC-20W_7.5x12.8mm_P1.27mm, symbol 74xx:74LS245
- added unit 1 of U9
- added unit 2 of U9
- added U? (x3): MAX3814, symbol VGA~V11-cache:MAX3814
- R23, R24: value 200 -> 10k
Connections:
- net labels added: +12V, AD0, AD1, AD10, AD11, AD12, AD13, AD14, AD15, AD16, AD17, AD18, AD19, AD2, AD20, AD21, AD22, AD23, AD24, AD25, AD26, AD27, AD28, AD29, AD3, AD30, AD31, AD4, AD5, AD6, AD7, AD8, AD9, AUD, CFG0, CFG1, CS1FX*, CS3FX*, CSEL, DA0, DA1, DA2, DASP*, DBEN*, DD0, DD1, DD10, DD11, DD12, DD13, DD14, DD15, DD2, DD3, DD4, DD5, DD6, DD7, DD8, DD9, DDIR, DDMARQ, DIOR*, DIORDY, DIOW*, DMACK*, DMARQ, DRDY*, FAD0, FAD1, FAD10, FAD11, FAD12, FAD13, FAD14, FAD15, FAD16, FAD17, FAD18, FAD19, FAD2, FAD20, FAD21, FAD22, FAD23, FAD24, FAD25, FAD26, FAD27, FAD28, FAD29, FAD3, FAD30, FAD31, FAD4, FAD5, FAD6, FAD7, FAD8, FAD9, FBDIR, FBEN, FCDIR, FCS1FX*, FCS3FX*, FDIOR*, FDIOW*, FIRQ0, FIRQ1, FIRQ10, FIRQ2, FIRQ3, FIRQ4, FIRQ5, FIRQ6, FIRQ7, FIRQ8, FIRQ9, FIRQS, FRCLK0N, FRCLK0P, FRD, FRDAT0N, FRDAT0P, FRDAT1N, FRDAT1P, FRDAT2N, FRDAT2P, FRDY*, FSEL0, FSEL1, FSEL2, FSEL3, FTCLK0N, FTCLK0P, FTDAT0N, FTDAT0P, FTDAT1N, FTDAT1P, FTDAT2N, FTDAT2P, INTRQ, IOCS16*, IRQ10, IRQ11, IRQ12, IRQ15, IRQ2, IRQ3, IRQ4, IRQ5, IRQ6, IRQ7, PDIAG, RCLK0N, RCLK0P, RD, RDAT0N, RDAT0P, RDAT1N, RDAT1P, RDAT2N, RDAT2P, RESET*, SEL0, SEL1, SEL2, SEL3, TCLK0N, TCLK0P, TDAT0N, TDAT0P, TDAT1N, TDAT1P, TDAT2N, TDAT2P, VCC_CF
- net labels removed: 8MH18Hz, A0, A1, A10, A11, A12, A13, A14, A15, A16, A17, A18, A19, A2, A20, A21, A22, A23, A24, A25, A26, A3, A4, A5, A6, A7, A8, A9, D0, D1, D10, D11, D12, D13, D14, D15, D2, D3, D4, D5, D6, D7, D8, D9, FA0, FA1, FA10, FA11, FA12, FA13, FA14, FA15, FA16, FA17, FA18, FA19, FA2, FA20, FA21, FA22, FA23, FA24, FA25, FA26, FA3, FA4, FA5, FA6, FA7, FA8, FA9, FD0, FD1, FD10, FD11, FD12, FD13, FD14, FD15, FD2, FD3, FD4, FD5, FD6, FD7, FD8, FD9, FDBE*, FMEMCS16, FSBHE, FWR*, MEMCS16*, PMODA0, PMODA1, PMODA2, PMODA3, PMODA4, PMODA5, PMODA6, PMODA7, PMODB0, PMODB1, PMODB2, PMODB3, RD*, SBHE, WR*
- wire segments 697 -> 838
- no-connect marks 13 -> 63
Other:
- moved on the sheet: C1, C10, C11, C2, C3, C4, C5, C6, C7, D1, J2, R1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
