File: ISA/ISA_FPGA/_autosave-ISA_FPGA_v2.sch (KiCad schematic (older format))
At the start: 127 parts, among them J1 Bus_ISA_16bit, J2 DE15, J3 AudioJack2, P1 CONN_5X2, P2 CONN_2, P3 CONN_5X2, P4 CONN_7, P5 CONN_6, P6 CONN_2X2, P7 CONN_7, P8 CONN_2, U1 74LVC245, U10 74LVC245, U11 74LVC244, U12 74LVC257, U13 CONN_6x2, U14 LM3940, U15 74LVC138, U16 LM386, U17 74LVC574, U18 74LVC257, U19 CONN_20X2, U2 74LVC245, U20 74LVC573, U21 74LVC245, U22 74LVC245, U3 74LVC245, U4 74LVC257, U5 74LVC245, U6 74LVC245, U7 CONN_32X2, U8 CONN_32X2, U9 74LVC06, X1 MINI_DIN_6, X2 MINI_DIN_6

Commit message: Petajon - update
Parts:
- removed J2: DE15, Connector_Dsub:DSUB-15-HD_Female_Horizontal_P2.29x1.98mm_EdgePinOffset3.03mm_Housed_MountingHolesOffset4.94mm, symbol VGA~V11-cache:DE15
- removed P1: CONN_5X2, Connector_PinHeader_2.54mm:PinHeader_2x05_P2.54mm_Vertical, symbol VGA~V11-cache:CONN_5X2
- removed R1, R5, R9: 510, Resistor_THT:R_Axial_DIN0207_L6.3mm_D2.5mm_P7.62mm_Horizontal, symbol VGA~V11-cache:R
- removed R10, R2, R6: 1k, Resistor_THT:R_Axial_DIN0207_L6.3mm_D2.5mm_P7.62mm_Horizontal, symbol VGA~V11-cache:R
- removed R11, R3, R7: 2k, Resistor_THT:R_Axial_DIN0207_L6.3mm_D2.5mm_P7.62mm_Horizontal, symbol VGA~V11-cache:R
- removed R12, R4, R8: 4k, Resistor_THT:R_Axial_DIN0207_L6.3mm_D2.5mm_P7.62mm_Horizontal, symbol VGA~V11-cache:R
- removed R13, R14: 100, Resistor_THT:R_Axial_DIN0207_L6.3mm_D2.5mm_P7.62mm_Horizontal, symbol VGA~V11-cache:R
- removed R? (x8): 200, Resistor_THT:R_Axial_DIN0207_L6.3mm_D2.5mm_P7.62mm_Horizontal, symbol VGA_V11-cache:R
- removed U12, U18, U4: 74LVC257, Package_SO:SOIC-16W_7.5x10.3mm_P1.27mm, symbol 74xx:74LS257
- removed U? (x2): MAX3814, symbol VGA~V11-cache:MAX3814
- added D2: ZPDxx, Diode_THT:D_DO-35_SOD27_P10.16mm_Horizontal, symbol Diode:ZPDxx
- added J2: HDMI_A, Connector_HDMI:HDMI_A_Contact_Technology_HDMI-19APL2_Horizontal, symbol Connector:HDMI_A
- added R10: 27k, Resistor_THT:R_Axial_DIN0207_L6.3mm_D2.5mm_P7.62mm_Horizontal, symbol VGA_V11-cache:R
- added R11, R12: 1k5, Resistor_THT:R_Axial_DIN0207_L6.3mm_D2.5mm_P7.62mm_Horizontal, symbol VGA_V11-cache:R
- added R13: 100k, Resistor_THT:R_Axial_DIN0207_L6.3mm_D2.5mm_P7.62mm_Horizontal, symbol VGA_V11-cache:R
- added R9: 10k, Resistor_THT:R_Axial_DIN0207_L6.3mm_D2.5mm_P7.62mm_Horizontal, symbol VGA_V11-cache:R
- added unit 6 of U9
- U12, U18, U4: renamed from U?; footprint (none) -> Package_QFP:TQFP-32_7x7mm_P0.8mm
- gave numbers to parts that had none: 8
Connections:
- net labels added: FINT, FINTA, FRCLK0N, FRCLK0P, FRDAT0N, FRDAT0P, FRDAT1N, FRDAT1P, FRDAT2N, FRDAT2P, FTCLK0N, FTCLK0P, FTDAT0N, FTDAT0P, FTDAT1N, FTDAT1P, FTDAT2N, FTDAT2P, INT*, INTA, RCLK0N, RCLK0P, RDAT0N, RDAT0P, RDAT1N, RDAT1P, RDAT2N, RDAT2P, VCC12
- net labels removed: +12V, BLUE0, BLUE1, BLUE2, BLUE3, CLK1N, CLK1P, CLK2N, CLK2P, DAT3N, DAT3P, DAT4N, DAT4P, DAT5N, DAT5P, DAT6N, DAT6P, DAT7N, DAT7P, DAT8N, DAT8P, FCLK0N, FCLK0P, FCLK1N, FCLK1P, FCLK2N, FCLK2P, FDAT0N, FDAT0P, FDAT1N, FDAT1P, FDAT2N, FDAT2P, FDAT3N, FDAT3P, FDAT4N, FDAT4P, FDAT5N, FDAT5P, FDAT6N, FDAT6P, FDAT7N, FDAT7P, FDAT8N, FDAT8P, FIRQ0, FIRQ1, FIRQ2, FIRQ3, FIRQ4, FIRQ5, FIRQ6, FIRQ7, FIRQ8, FIRQ9, FIRQS, GREEN0, GREEN1, GREEN2, GREEN3, HS, IRQ10, IRQ11, IRQ12, IRQ15, IRQ3, IRQ4, IRQ5, IRQ6, IRQ7, RED0, RED1, RED2, RED3, VS
- wire segments 906 -> 812
- no-connect marks 63 -> 45
Other:
- moved on the sheet: R1, R2, R3, R4, R5, R6, R7, R8, RR1, U12, U13, U18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
