File: FAL6567/trunk/KiCad/FAL6567i.kicad_pcb (KiCad board)
At the start: 2 copper layers, 98 x 150.1 mm, 37 parts, among them IC1 74245DW, IC2 74LVC245, IC3 74LVC245, IC4 74LVC245, IC6 REG1117F, IC9 74ALS573, J1 HDMI_A_1.4_Shielded, U1 MAX3814, U7 74LS06N

Commit message: FAL6567 - update
Parts:
- removed IC1: 74245DW, Package_DIP:DIP-20_W7.62mm
- removed IC2, IC3, IC4: 74LVC245, Package_DIP:DIP-20_W7.62mm
- removed IC6: REG1117F, FAL6567h:DD-3
- removed IC9: 74ALS573, Package_DIP:DIP-20_W7.62mm
- added IC5: REG1117F, Package_TO_SOT_THT:TO-262-3-1EP_Horizontal_TabDown, F.Cu at (132.6, 61.7)
- added R10: 1k, FAL6567h:0204_7, F.Cu at (84.8, 115.3)
- added R11: 470, FAL6567h:0204_7, F.Cu at (84.8, 112.8)
- added R13: 220, FAL6567h:0204_7, F.Cu at (84.8, 110.2)
- added R9: 2k2, FAL6567h:0204_7, F.Cu at (84.8, 117.9)
- added U1: 74LS245, Package_DIP:DIP-20_W7.62mm, F.Cu at (113.0, 123.2)
- added U2: 74LS245, Package_DIP:DIP-20_W7.62mm, F.Cu at (97.8, 87.6)
- added U3: 74LS245, Package_DIP:DIP-20_W7.62mm, F.Cu at (113.0, 87.6)
- added U4: 74LS245, Package_DIP:DIP-20_W7.62mm, F.Cu at (97.8, 123.2)
- added U9: 74ALS573, Package_DIP:DIP-20_W7.62mm, F.Cu at (135.6, 147.3)
- U7: value 74LS06N -> 74LS06
- moved R8 22.8 mm to (91.7, 71.6), turned to 90 degrees
- moved C3 22.1 mm to (139.4, 142.2)
- moved C1 11.0 mm to (80.8, 43.2), turned to -90 degrees
- moved R5 6.65 mm to (91.9, 53.8), turned to -90 degrees
- moved C2 5.61 mm to (101.6, 116.8)
- moved R1 4.68 mm to (115.6, 62.0)
- moved R2 4.68 mm to (115.6, 64.5)
- moved R6 3.31 mm to (86.9, 61.0), turned to -90 degrees
- moved J1 3.05 mm to (97.3, 51.8)
- moved R4 2.79 mm to (100.8, 80.5)
- moved R7 0.80 mm to (86.6, 71.9), turned to -90 degrees
- moved U7 0.76 mm to (80.0, 154.9)
- renumbered U1 to U10
Connections:
- net Net-(U$1-Pad22) renamed /nc
- C5 pad 1: +3V3 -> +5V
- D2 pad A: +3V3 -> +5V
- J1 pad 14: Net-(J1-Pad14) -> unconnected-(J1-Pad14)
- J1 pad 18: +3V3 -> +5V
- J1 pad 19: Net-(J1-Pad19) -> unconnected-(J1-Pad19)
- R1 pad 2: +3V3 -> +5V
- R2 pad 2: +3V3 -> +5V
- U$1 pad 14: /COLOR -> unconnected-(U$1-Pad14)
- U$1 pad 21: /VCLRCLK -> unconnected-(U$1-Pad21)
- U$1 pad 40: +3V3 -> +5V
- U$2 pad 15: Net-(U$2-Pad15) -> unconnected-(U$2-Pad15)
- U$2 pad 16: Net-(U$2-Pad16) -> unconnected-(U$2-Pad16)
- U$2 pad 18: Net-(U$2-Pad18) -> /RESET
- U$2 pad 34: /RESET -> /IRQ
- U$2 pad 36: Net-(U$2-Pad36) -> /LUMA0
- U$2 pad 37: /IRQ -> /LUMA1
- U$2 pad 38: Net-(U$2-Pad38) -> /LUMA2
- U$2 pad 39: Net-(U$2-Pad39) -> /LUMA3
- U10 pad 1: Net-(U1-Pad1) -> unconnected-(U10-Pad1)
- U10 pad 17: Net-(U1-Pad17) -> unconnected-(U10-Pad17)
- U10 pad 24: Net-(U1-Pad24) -> unconnected-(U10-Pad24)
- U10 pad 8: Net-(U1-Pad8) -> unconnected-(U10-Pad8)
- U7 pad 10: Net-(U7-Pad10) -> unconnected-(U7-Pad10)
- U7 pad 12: Net-(U7-Pad12) -> unconnected-(U7-Pad12)
- U7 pad 14: +3V3 -> +5V
- U7 pad 6: Net-(U7-Pad6) -> unconnected-(U7-Pad6)
- U7 pad 8: Net-(U7-Pad8) -> unconnected-(U7-Pad8)
Routing:
- net +3V3: track 606.0 -> 0.00 mm, vias 2 -> 0
- net GND: track 489.2 -> 0.00 mm
- net /A1: track 117.0 -> 0.00 mm
- net /D11: track 115.2 -> 0.00 mm
- net /A3: track 108.5 -> 0.00 mm
- net /AEC: track 107.9 -> 0.00 mm, vias 3 -> 0
- net /A0: track 107.3 -> 0.00 mm
- net /D1P: track 101.5 -> 0.00 mm
- net Net-(U$1-Pad8): track 99.6 -> 0.00 mm
- net /BA: track 97.9 -> 0.00 mm
- net /A2: track 96.3 -> 0.00 mm
- net /RAS: track 96.1 -> 0.00 mm
- net /D0P: track 94.9 -> 0.00 mm
- net /D1N: track 92.5 -> 0.00 mm
- net /D2N: track 91.1 -> 0.00 mm
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Other:
- net class Default removed
