File: RF65816SBC/Clkgen2.kicad_sch (KiCad schematic)
At the start: 12 parts, among them U20 G65SC22P, U21 74ACT163, U22 74ACT163, U23 74ACT74, U24 74ACT14, U25 74HC4046

Commit message: RF65816 - update
Parts:
- added R?: 4k7, symbol Device:R
- U21, U22: value 74ACT163 -> 74AC163
- U23: value 74ACT74 -> 74AC74
- U24: value 74ACT14 -> 74AC14
Connections:
- net +5V: no longer U20.20 (VDD), U20.8 (PA6), U21.16 (VCC), U22.16 (VCC), U22.5 (D2), U23.1 (~{R}), U23.10 (~{S}), U23.13 (~{R}), U23.14 (VCC), U23.4 (~{S}), U24.14 (VCC), U25.16 (VDD)
- new net: U23.10 (~{S}), U23.13 (~{R})
- new net: U23.1 (~{R}), U23.4 (~{S})
- new net +3.3V: R?.1, U20.20 (VDD), U21.16 (VCC), U22.16 (VCC), U23.14 (VCC), U24.14 (VCC), U25.16 (VDD)
- new net P6: R?.2, U20.8 (PA6), U22.5 (D2)
