File: RF65816SBC/ClkGen.kicad_sch (KiCad schematic)
At the start: 9 parts, among them U1 74AC04

Commit message: RF65816SBC - update
Parts:
- gave numbers to parts that had none: 3
Changed lines of the file:
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@@
   (symbol (lib_id "MyLib:G65SC22P") (at 116.84 110.49 0) (unit 1)
     (in_bom yes) (on_board yes) (fields_autoplaced)
-    (property "Reference" "U?" (id 0) (at 116.84 110.49 0)
+    (property "Reference" "U7" (id 0) (at 116.84 110.49 0)
       (effects (font (size 1.27 1.27)) hide)
     )
@@
   (symbol (lib_id "Timer_PLL:ICS525R-02") (at 179.07 74.93 0) (unit 1)
     (in_bom yes) (on_board yes) (fields_autoplaced)
-    (property "Reference" "U?" (id 0) (at 181.0894 112.5204 0)
+    (property "Reference" "U6" (id 0) (at 181.0894 112.5204 0)
       (effects (font (size 1.27 1.27)) (justify left))
     )
@@
   (symbol (lib_id "MyLib:74F521") (at 66.04 134.62 0) (unit 1)
     (in_bom yes) (on_board yes) (fields_autoplaced)
-    (property "Reference" "U?" (id 0) (at 66.7894 118.271 0)
+    (property "Reference" "U8" (id 0) (at 66.7894 118.271 0)
       (effects (font (size 1.27 1.27)) (justify left))
     )
