File: RF65816SBC/RF65816SBC.kicad_sch (KiCad schematic)
At the start: 66 parts, among them U1 74AC04, U2 74AC08, U20 74AC245, U21 74AC245, U22 74AC245, U30 WM1-SRAM, U31 WM1-SRAM, U32 WM1-SRAM

Commit message: RF65816 - update
Parts:
- removed unit 5 of U1
- removed unit 6 of U1
- removed U?: 74ACT02, symbol 74xx:74LS02
- added U? (x2): 74AC04, symbol 74xx:74LS04
- added U?: 74AC08, symbol 74xx:74LS08
- U? (x2): value DS1813 -> DS1818
Connections:
- net RVDA is gone; now on net MVDA: U?.16 (O1a)
- net RVPA is gone; now on net MVPA: U?.14 (O2a)
- net +3.3V: now also R?.1, RN?.1 (common), U?.2 (VCC)
- net +5V: no longer R?.1, RN?.1 (common), U?.2 (VCC)
- net GND: now also R?.1
- net RA22: now also U?.11
- net RA23: now also U?.13
- net at U?.19 (CE): now also U?.6
- net MVDA: now reaches U?.23 (PIO23)
- net RED0 renamed MVPA
- net MVPA: no longer R?.1
- new net: U?.10, U?.4
- new net: U?.12, U?.5
- no-connect marks 24 -> 22

Commit message: RF65816SBC - update
Broken out Serial, SRAM, and VGA
Parts:
- removed C? (x7): 0.1u, symbol Device:C
- removed C?: 220u, Capacitor_THT:CP_Radial_D8.0mm_P3.80mm, symbol ISA_FPGA_v2-rescue:CP1-Device
- removed C?: 100u, Capacitor_THT:CP_Radial_D8.0mm_P3.80mm, symbol ISA_FPGA_v2-rescue:CP1-Device
- removed C?: 0.047u, Capacitor_THT:C_Disc_D3.8mm_W2.6mm_P2.50mm, symbol ISA_FPGA_v2-rescue:CP1-Device
- removed C?: 0.047u, Capacitor_THT:C_Disc_D5.0mm_W2.5mm_P5.00mm, symbol ISA_FPGA_v2-rescue:CP1-Device
- removed C?: 10u, Capacitor_THT:CP_Radial_D5.0mm_P2.50mm, symbol ISA_FPGA_v2-rescue:CP1-Device
- removed D?: DIODE, symbol pspice:DIODE
- removed J?: DB15_Female_HighDensity, symbol Connector:DB15_Female_HighDensity
- removed J?: Audio In, Connector_Audio:Jack_3.5mm_CUI_SJ1-3533NG_Horizontal, symbol Connector:AudioJack2
- removed J?: AudioJack2, Connector_Audio:Jack_3.5mm_CUI_SJ1-3533NG_Horizontal, symbol Connector:AudioJack2
- removed R? (x3): 1k, symbol Device:R
- removed R? (x3): 510, symbol Device:R
- removed R? (x2): 100, symbol Device:R
- removed R? (x3): 10k, symbol Device:R
- removed R? (x3): 3k3, symbol Device:R
- removed R? (x2): 2k, symbol Device:R
- removed R?: 220k, symbol Device:R
- removed R? (x2): 5k1, Resistor_THT:R_Axial_DIN0207_L6.3mm_D2.5mm_P7.62mm_Horizontal, symbol VGA_V11-cache:R
- removed R?: 10, Resistor_THT:R_Axial_DIN0207_L6.3mm_D2.5mm_P7.62mm_Horizontal, symbol VGA_V11-cache:R
- removed unit 1 of U1
- removed U20, U21, U22: 74AC245, symbol 74xx:74LS245
- removed U30, U31, U32: WM1-SRAM, symbol MyLib:WM1-SRAM
- removed U? (x3): 74AC139, symbol 74xx:74LS139
- removed U?: 74AC138, symbol 74xx:74LS138
- removed U?: VDIP2-32, Package_DIP:DIP-32_W15.24mm_Socket, symbol MyLib:VDIP2-32
- removed U?: LM741, symbol Amplifier_Operational:LM741
- removed U?: CModA7, symbol MyLib:CModA7
- removed U? (x2): 74AC04, symbol 74xx:74LS04
- removed U?: 74AC08, symbol 74xx:74LS08
- removed U?: LM386, Package_DIP:DIP-8_W7.62mm_Socket, symbol Amplifier_Audio:LM386
- removed U?: 74LVC245, symbol 74xx:74LS245
Connections:
- net IRQ renamed VIRQ
- no-connect marks 22 -> 5
Other:
- added sheet SRAM (SRAM.kicad_sch)
- added sheet SerialIO (SerialIO.kicad_sch)
- added sheet VGAIO (VGAIO.kicad_sch)
- note removed: "USB Host for keyboard / mouse"
- title: 65816 SBC -> 65816 SBC CPU
- moved on the sheet: C?, R?, RN?, U1B, U1C, U1G, U2E, U?

Commit message: RF65816SBC - update
Parts:
- removed U2: 74AC08, symbol 74xx:74LS08
- added U2: 74AC11, symbol 74xx:74LS11
- gave numbers to parts that had none: 7
Connections:
- net +3.3V: now also U2.14 (VCC), U2.4
- net CBE: now also U2.5
- net GND: now also U2.7 (GND)
- net IRQ6522: now also U2.13
- net IRQB: now also U2.12
- net MPH2: now also U2.3
- net VIRQ: now also U2.1
- net at U3.37 (PH2-IN): now also U2.6
- new net SIRQ: U2.2
Other:
- title: 65816 SBC CPU -> RF65816SBC CPU
