File: RF65816SBC/SRAM.kicad_sch (KiCad schematic)
At the start: 23 parts

Commit message: RF65816SBC - update
Parts:
- removed U?: 74AC08, symbol 74xx:74LS08
- added U2: 74AC11, symbol 74xx:74LS11
- gave numbers to parts that had none: 16
Connections:
- net at U58.19 (CE): now also U2.8
- net at U1.12: now also U2.11
- net at U1.10: now also U2.10, U2.9
Changed lines of the file:
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@@
   (junction (at 97.79 40.64) (diameter 0) (color 0 0 0 0)
   )
+  (junction (at 237.49 91.44) (diameter 0) (color 0 0 0 0)
+  )
   (junction (at 147.32 105.41) (diameter 0) (color 0 0 0 0)
   )
@@
     (stroke (width 0) (type default) (color 0 0 0 0))
   )
-  (wire (pts (xy 240.03 91.44) (xy 232.41 91.44))
+  (wire (pts (xy 240.03 91.44) (xy 237.49 91.44))
     (stroke (width 0) (type default) (color 0 0 0 0))
   )
@@
     (stroke (width 0) (type default) (color 0 0 0 0))
   )
+  (wire (pts (xy 232.41 93.98) (xy 237.49 93.98))
+    (stroke (width 0) (type default) (color 0 0 0 0))
+  )
   (bus (pts (xy 214.63 60.96) (xy 214.63 58.42))
     (stroke (width 0) (type default) (color 0 0 0 0))
@@
     (stroke (width 0) (type default) (color 0 0 0 0))
   )
+  (wire (pts (xy 237.49 91.44) (xy 232.41 91.44))
+    (stroke (width 0) (type default) (color 0 0 0 0))
+  )
   (wire (pts (xy 254 53.34) (xy 260.35 53.34))
     (stroke (width 0) (type default) (color 0 0 0 0))
@@
     (stroke (width 0) (type default) (color 0 0 0 0))
   )
+  (wire (pts (xy 237.49 91.44) (xy 237.49 93.98))
+    (stroke (width 0) (type default) (color 0 0 0 0))
+  )
   (wire (pts (xy 111.76 97.79) (xy 109.22 97.79))
     (stroke (width 0) (type default) (color 0 0 0 0))
@@
   (symbol (lib_id "74xx:74LS245") (at 50.8 48.26 0) (unit 1)
     (in_bom yes) (on_board yes) (fields_autoplaced)
-    (property "Reference" "U?" (id 0) (at 52.8194 29.3202 0)
+    (property "Reference" "U50" (id 0) (at 52.8194 29.3202 0)
       (effects (font (size 1.27 1.27)) (justify left))
     )
@@
   (symbol (lib_id "Device:C") (at 100.33 185.42 0) (unit 1)
     (in_bom yes) (on_board yes) (fields_autoplaced)
-    (property "Reference" "C?" (id 0) (at 103.251 184.5853 0)
+    (property "Reference" "C54" (id 0) (at 103.251 184.5853 0)
       (effects (font (size 1.27 1.27)) (justify left))
     )
@@
   (symbol (lib_id "Device:C") (at 69.85 185.42 0) (unit 1)
     (in_bom yes) (on_board yes) (fields_autoplaced)
-    (property "Reference" "C?" (id 0) (at 72.771 184.5853 0)
+    (property "Reference" "C50" (id 0) (at 72.771 184.5853 0)
       (effects (font (size 1.27 1.27)) (justify left))
     )
@@
   (symbol (lib_id "74xx:74LS139") (at 251.46 134.62 0) (unit 3)
     (in_bom yes) (on_board yes)
-    (property "Reference" "U?" (id 0) (at 257.302 133.7853 0)
+    (property "Reference" "U53" (id 0) (at 257.302 133.7853 0)
       (effects (font (size 1.27 1.27)) (justify left))
     )
@@
   (symbol (lib_id "74xx:74LS245") (at 50.8 99.06 0) (unit 1)
     (in_bom yes) (on_board yes)
-    (property "Reference" "U?" (id 0) (at 57.15 80.01 0)
+    (property "Reference" "U51" (id 0) (at 57.15 80.01 0)
       (effects (font (size 1.27 1.27)) (justify left))
     )
@@
   (symbol (lib_id "74xx:74LS04") (at 81.28 154.94 90) (unit 1)
     (in_bom yes) (on_board yes) (fields_autoplaced)
-    (property "Reference" "U?" (id 0) (at 85.852 154.1053 90)
+    (property "Reference" "U1" (id 0) (at 85.852 154.1053 90)
       (effects (font (size 1.27 1.27)) (justify right))
     )
@@
   (symbol (lib_id "MyLib:WM1-SRAM") (at 147.32 71.12 0) (unit 1)
     (in_bom yes) (on_board yes) (fields_autoplaced)
-    (property "Reference" "U?" (id 0) (at 151.8794 40.801 0)
+    (property "Reference" "U56" (id 0) (at 151.8794 40.801 0)
       (effects (font (size 1.27 1.27)) (justify left))
     )
@@
   (symbol (lib_id "74xx:74LS139") (at 97.79 129.54 0) (unit 1)
     (in_bom yes) (on_board yes) (fields_autoplaced)
-    (property "Reference" "U?" (id 0) (at 97.79 120.7602 0))
+    (property "Reference" "U53" (id 0) (at 97.79 120.7602 0))
     (property "Value" "74LVC139" (id 1) (at 97.79 123.2971 0))
     (property "Footprint" "" (id 2) (at 97.79 129.54 0)
@@
   (symbol (lib_id "74xx:74LS139") (at 148.59 130.81 0) (unit 2)
     (in_bom yes) (on_board yes) (fields_autoplaced)
-    (property "Reference" "U?" (id 0) (at 148.59 122.0302 0))
+    (property "Reference" "U53" (id 0) (at 148.59 122.0302 0))
     (property "Value" "74LVC139" (id 1) (at 148.59 124.5671 0))
     (property "Footprint" "" (id 2) (at 148.59 130.81 0)
@@
   (symbol (lib_id "Device:C") (at 107.95 185.42 0) (unit 1)
     (in_bom yes) (on_board yes) (fields_autoplaced)
-    (property "Reference" "C?" (id 0) (at 110.871 184.5853 0)
+    (property "Reference" "C58" (id 0) (at 110.871 184.5853 0)
       (effects (font (size 1.27 1.27)) (justify left))
     )
@@
     (pin "2")
   )
+  (symbol (lib_id "74xx:74LS11") (at 224.79 93.98 0) (mirror y) (unit 3)
+    (in_bom yes) (on_board yes) (fields_autoplaced)
+    (property "Reference" "U2" (id 0) (at 224.79 86.4702 0))
+    (property "Value" "74AC11" (id 1) (at 224.79 89.0071 0))
+    (property "Footprint" "" (id 2) (at 224.79 93.98 0)
+      (effects (font (size 1.27 1.27)) hide)
+    )
+    (property "Datasheet" "http://www.ti.com/lit/gpn/sn74LS11" (id 3) (at 224.79 93.98 0)
+      (effects (font (size 1.27 1.27)) hide)
+    )
+    (pin "1")
+    (pin "12")
+    (pin "13")
+    (pin "2")
+    (pin "3")
+    (pin "4")
+    (pin "5")
+    (pin "6")
+    (pin "10")
+    (pin "11")
+    (pin "8")
+    (pin "9")
+    (pin "14")
+    (pin "7")
+  )
   (symbol (lib_id "power:+3.3V") (at 50.8 78.74 0) (unit 1)
     (in_bom yes) (on_board yes) (fields_autoplaced)
@@
   (symbol (lib_id "74xx:74LS245") (at 241.3 60.96 0) (unit 1)
     (in_bom yes) (on_board yes) (fields_autoplaced)
-    (property "Reference" "U?" (id 0) (at 243.3194 42.0202 0)
+    (property "Reference" "U58" (id 0) (at 243.3194 42.0202 0)
       (effects (font (size 1.27 1.27)) (justify left))
     )
@@
   (symbol (lib_id "74xx:74LS04") (at 246.38 102.87 0) (mirror y) (unit 6)
     (in_bom yes) (on_board yes) (fields_autoplaced)
-    (property "Reference" "U?" (id 0) (at 246.38 95.3602 0))
+    (property "Reference" "U1" (id 0) (at 246.38 95.3602 0))
     (property "Value" "74AC04" (id 1) (at 246.38 97.8971 0))
     (property "Footprint" "" (id 2) (at 246.38 102.87 0)
@@
   (symbol (lib_id "Device:C") (at 92.71 185.42 0) (unit 1)
     (in_bom yes) (on_board yes) (fields_autoplaced)
-    (property "Reference" "C?" (id 0) (at 95.631 184.5853 0)
+    (property "Reference" "C53" (id 0) (at 95.631 184.5853 0)
       (effects (font (size 1.27 1.27)) (justify left))
     )
@@
     (pin "1")
   )
-  (symbol (lib_id "74xx:74LS08") (at 224.79 93.98 0) (mirror y) (unit 2) (convert 2)
-    (in_bom yes) (on_board yes) (fields_autoplaced)
-    (property "Reference" "U?" (id 0) (at 224.79 86.4702 0))
-    (property "Value" "74AC08" (id 1) (at 224.79 89.0071 0))
-    (property "Footprint" "" (id 2) (at 224.79 93.98 0)
-      (effects (font (size 1.27 1.27)) hide)
-    )
-    (property "Datasheet" "http://www.ti.com/lit/gpn/sn74LS08" (id 3) (at 224.79 93.98 0)
-      (effects (font (size 1.27 1.27)) hide)
-    )
-    (pin "1")
-    (pin "2")
-    (pin "3")
-    (pin "4")
-    (pin "5")
-    (pin "6")
-    (pin "10")
-    (pin "8")
-    (pin "9")
-    (pin "11")
-    (pin "12")
-    (pin "13")
-    (pin "14")
-    (pin "7")
-  )
   (symbol (lib_id "power:GND") (at 146.05 105.41 0) (unit 1)
     (in_bom yes) (on_board yes) (fields_autoplaced)
@@
   (symbol (lib_id "74xx:74LS138") (at 199.39 139.7 0) (unit 1)
     (in_bom yes) (on_board yes) (fields_autoplaced)
-    (property "Reference" "U?" (id 0) (at 201.4094 125.8402 0)
+    (property "Reference" "U54" (id 0) (at 201.4094 125.8402 0)
       (effects (font (size 1.27 1.27)) (justify left))
     )
@@
   (symbol (lib_id "74xx:74LS245") (at 50.8 149.86 0) (unit 1)
     (in_bom yes) (on_board yes) (fields_autoplaced)
-    (property "Reference" "U?" (id 0) (at 52.8194 130.9202 0)
+    (property "Reference" "U52" (id 0) (at 52.8194 130.9202 0)
       (effects (font (size 1.27 1.27)) (justify left))
     )
@@
   (symbol (lib_id "MyLib:WM1-SRAM") (at 97.79 71.12 0) (unit 1)
     (in_bom yes) (on_board yes) (fields_autoplaced)
-    (property "Reference" "U?" (id 0) (at 102.3494 40.801 0)
+    (property "Reference" "U55" (id 0) (at 102.3494 40.801 0)
       (effects (font (size 1.27 1.27)) (justify left))
     )
@@
   (symbol (lib_id "Device:C") (at 85.09 185.42 0) (unit 1)
     (in_bom yes) (on_board yes) (fields_autoplaced)
-    (property "Reference" "C?" (id 0) (at 88.011 184.5853 0)
+    (property "Reference" "C52" (id 0) (at 88.011 184.5853 0)
       (effects (font (size 1.27 1.27)) (justify left))
     )
@@
   (symbol (lib_id "Device:C") (at 77.47 185.42 0) (unit 1)
     (in_bom yes) (on_board yes) (fields_autoplaced)
-    (property "Reference" "C?" (id 0) (at 80.391 184.5853 0)
+    (property "Reference" "C51" (id 0) (at 80.391 184.5853 0)
       (effects (font (size 1.27 1.27)) (justify left))
     )
@@
   (symbol (lib_id "MyLib:WM1-SRAM") (at 195.58 71.12 0) (unit 1)
     (in_bom yes) (on_board yes) (fields_autoplaced)
-    (property "Reference" "U?" (id 0) (at 200.1394 40.801 0)
+    (property "Reference" "U57" (id 0) (at 200.1394 40.801 0)
       (effects (font (size 1.27 1.27)) (justify left))
     )
@@
   (symbol (lib_id "74xx:74LS04") (at 247.65 91.44 0) (mirror y) (unit 5)
     (in_bom yes) (on_board yes) (fields_autoplaced)
-    (property "Reference" "U?" (id 0) (at 247.65 83.9302 0))
+    (property "Reference" "U1" (id 0) (at 247.65 83.9302 0))
     (property "Value" "74AC04" (id 1) (at 247.65 86.4671 0))
     (property "Footprint" "" (id 2) (at 247.65 91.44 0)
