File: RF65816SBC/SerialIO.kicad_sch (KiCad schematic)
At the start: 22 parts

Commit message: RF65816SBC - update
Parts:
- gave numbers to parts that had none: 4
Connections:
- net IRQ renamed SIRQ
Changed lines of the file:
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@@
+    (stroke (width 0) (type default) (color 0 0 0 0))
+  )
+  (wire (pts (xy 55.88 92.71) (xy 64.77 92.71))
     (stroke (width 0) (type default) (color 0 0 0 0))
   )
@@
     (stroke (width 0) (type default) (color 0 0 0 0))
   )
+  (wire (pts (xy 54.61 90.17) (xy 64.77 90.17))
+    (stroke (width 0) (type default) (color 0 0 0 0))
+  )
   (wire (pts (xy 64.77 39.37) (xy 58.42 39.37))
     (stroke (width 0) (type default) (color 0 0 0 0))
@@
     (stroke (width 0) (type default) (color 0 0 0 0))
   )
-  (wire (pts (xy 64.77 87.63) (xy 57.15 87.63))
-    (stroke (width 0) (type default) (color 0 0 0 0))
-  )
   (wire (pts (xy 227.33 115.57) (xy 227.33 113.03))
     (stroke (width 0) (type default) (color 0 0 0 0))
   )
-  (wire (pts (xy 64.77 85.09) (xy 58.42 85.09))
-    (stroke (width 0) (type default) (color 0 0 0 0))
-  )
   (wire (pts (xy 133.35 165.1) (xy 152.4 165.1))
     (stroke (width 0) (type default) (color 0 0 0 0))
@@
     (stroke (width 0) (type default) (color 0 0 0 0))
   )
+  (wire (pts (xy 55.88 85.09) (xy 64.77 85.09))
+    (stroke (width 0) (type default) (color 0 0 0 0))
+  )
   (wire (pts (xy 229.87 115.57) (xy 227.33 115.57))
     (stroke (width 0) (type default) (color 0 0 0 0))
@@
     (stroke (width 0) (type default) (color 0 0 0 0))
   )
+  (wire (pts (xy 55.88 87.63) (xy 64.77 87.63))
+    (stroke (width 0) (type default) (color 0 0 0 0))
+  )
   (wire (pts (xy 218.44 107.95) (xy 215.9 107.95))
     (stroke (width 0) (type default) (color 0 0 0 0))
@@
     (stroke (width 0) (type default) (color 0 0 0 0))
   )
-  (wire (pts (xy 64.77 92.71) (xy 58.42 92.71))
-    (stroke (width 0) (type default) (color 0 0 0 0))
-  )
   (wire (pts (xy 144.78 143.51) (xy 138.43 143.51))
     (stroke (width 0) (type default) (color 0 0 0 0))
@@
     (stroke (width 0) (type default) (color 0 0 0 0))
   )
-  (wire (pts (xy 52.07 82.55) (xy 64.77 82.55))
+  (wire (pts (xy 55.88 82.55) (xy 64.77 82.55))
     (stroke (width 0) (type default) (color 0 0 0 0))
   )
@@
     (stroke (width 0) (type default) (color 0 0 0 0))
   )
-  (wire (pts (xy 64.77 90.17) (xy 58.42 90.17))
-    (stroke (width 0) (type default) (color 0 0 0 0))
-  )
   (wire (pts (xy 142.24 97.79) (xy 142.24 100.33))
     (stroke (width 0) (type default) (color 0 0 0 0))
@@
   (label "CD4" (at 87.63 46.99 0)
     (effects (font (size 1.27 1.27)) (justify left bottom))
+  )
+  (global_label "RRW" (shape input) (at 54.61 90.17 180) (fields_autoplaced)
+    (effects (font (size 1.27 1.27)) (justify right))
+    (property "Intersheet References" "${INTERSHEET_REFS}" (id 0) (at 48.2055 90.0906 0)
+      (effects (font (size 1.27 1.27)) (justify right) hide)
+    )
+  )
+  (global_label "SIRQ" (shape output) (at 55.88 85.09 180) (fields_autoplaced)
+    (effects (font (size 1.27 1.27)) (justify right))
+    (property "Intersheet References" "${INTERSHEET_REFS}" (id 0) (at 49.0521 85.0106 0)
+      (effects (font (size 1.27 1.27)) (justify right) hide)
+    )
+  )
+  (global_label "MVDA" (shape input) (at 55.88 92.71 180) (fields_autoplaced)
+    (effects (font (size 1.27 1.27)) (justify right))
+    (property "Intersheet References" "${INTERSHEET_REFS}" (id 0) (at 48.5683 92.6306 0)
+      (effects (font (size 1.27 1.27)) (justify right) hide)
+    )
   )
   (global_label "DATA BUS" (shape bidirectional) (at 90.17 25.4 180) (fields_autoplaced)
@@
     )
   )
+  (global_label "MPH2" (shape input) (at 55.88 82.55 180) (fields_autoplaced)
+    (effects (font (size 1.27 1.27)) (justify right))
+    (property "Intersheet References" "${INTERSHEET_REFS}" (id 0) (at 48.2055 82.4706 0)
+      (effects (font (size 1.27 1.27)) (justify right) hide)
+    )
+  )
   (global_label "ADDR BUS" (shape bidirectional) (at 52.07 30.48 180) (fields_autoplaced)
     (effects (font (size 1.27 1.27)) (justify right))
@@
     )
   )
+  (global_label "MVPA" (shape input) (at 55.88 87.63 180) (fields_autoplaced)
+    (effects (font (size 1.27 1.27)) (justify right))
+    (property "Intersheet References" "${INTERSHEET_REFS}" (id 0) (at 48.5683 87.5506 0)
+      (effects (font (size 1.27 1.27)) (justify right) hide)
+    )
+  )
   (symbol (lib_id "ISA_FPGA_v2-rescue:CP1-Device") (at 104.14 124.46 0) (unit 1)
     (in_bom yes) (on_board yes)
@@
   (symbol (lib_id "Amplifier_Operational:LM741") (at 237.49 113.03 0) (unit 1)
     (in_bom yes) (on_board yes)
-    (property "Reference" "U?" (id 0) (at 238.76 107.95 0))
+    (property "Reference" "U34" (id 0) (at 238.76 107.95 0))
     (property "Value" "LM741" (id 1) (at 240.03 105.41 0))
     (property "Footprint" "" (id 2) (at 238.76 111.76 0)
@@
   (symbol (lib_id "MyLib:VDIP2-32") (at 143.51 73.66 0) (mirror y) (unit 1)
     (in_bom yes) (on_board yes) (fields_autoplaced)
-    (property "Reference" "U?" (id 0) (at 138.9506 49.691 0)
+    (property "Reference" "U32" (id 0) (at 138.9506 49.691 0)
       (effects (font (size 1.27 1.27)) (justify left))
     )
@@
   (symbol (lib_id "MyLib:CModA7") (at 73.66 64.77 0) (unit 1)
     (in_bom yes) (on_board yes) (fields_autoplaced)
-    (property "Reference" "U?" (id 0) (at 75.565 31.911 0))
+    (property "Reference" "U31" (id 0) (at 75.565 31.911 0))
     (property "Value" "CModA7" (id 1) (at 75.565 34.4479 0))
     (property "Footprint" "" (id 2) (at 74.93 31.75 0)
@@
   (symbol (lib_id "Amplifier_Audio:LM386") (at 135.89 135.89 0) (unit 1)
     (in_bom yes) (on_board yes)
-    (property "Reference" "U?" (id 0) (at 144.6276 134.7216 0)
-      (effects (font (size 1.27 1.27)) (justify left))
-    )
+    (property "Reference" "U33" (id 0) (at 144.6276 134.7216 0)
+      (effects (font (size 1.27 1.27)) (justify left))
+    )
