File: RF65816SBC/VGAIO.kicad_sch (KiCad schematic)
At the start: 17 parts

Commit message: RF65816SBC - update
Parts:
- gave numbers to parts that had none: 1
Changed lines of the file:
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@@
   (symbol (lib_id "MyLib:CModA7") (at 93.98 74.93 0) (unit 1)
     (in_bom yes) (on_board yes) (fields_autoplaced)
-    (property "Reference" "U?" (id 0) (at 95.885 42.071 0))
+    (property "Reference" "U40" (id 0) (at 95.885 42.071 0))
     (property "Value" "CModA7" (id 1) (at 95.885 44.6079 0))
     (property "Footprint" "" (id 2) (at 95.25 41.91 0)
