File: ISA/ISA65816/Clkgen.kicad_sch (KiCad schematic)
At the start: 15 parts

Commit message: ISA65816 - update
Parts:
- removed U?: 74AC04, symbol 74xx:74LS04
- removed U?: G65SC22P, FAL65816_Audio:DIP-40, symbol MyLib:G65SC22P
- removed U?: 74LVC521, symbol MyLib:74F521
- removed U?: 74LVC670, symbol 74xx:74LS670
- added C1, C14, C15, C31: 0.1u, symbol Device:C
- added C32: 0.047u, Capacitor_THT:C_Disc_D3.8mm_W2.6mm_P2.50mm, symbol ISA_FPGA_v2-rescue:CP1-Device
- added C33: 100u, Capacitor_THT:CP_Radial_D8.0mm_P3.80mm, symbol ISA_FPGA_v2-rescue:CP1-Device
- added C34: 10u, Capacitor_THT:CP_Radial_D5.0mm_P2.50mm, symbol ISA_FPGA_v2-rescue:CP1-Device
- added C35: 220u, Capacitor_THT:CP_Radial_D8.0mm_P3.80mm, symbol ISA_FPGA_v2-rescue:CP1-Device
- added C36: 0.047u, Capacitor_THT:C_Disc_D5.0mm_W2.5mm_P5.00mm, symbol ISA_FPGA_v2-rescue:CP1-Device
- added J2: Audio In, Connector_Audio:Jack_3.5mm_CUI_SJ1-3533NG_Horizontal, symbol Connector:AudioJack2
- added J3: AudioJack2, Connector_Audio:Jack_3.5mm_CUI_SJ1-3533NG_Horizontal, symbol Connector:AudioJack2
- added R2, R3, R5: 10k, Resistor_THT:R_Axial_DIN0309_L9.0mm_D3.2mm_P12.70mm_Horizontal, symbol Device:R
- added R4: 220k, Resistor_THT:R_Axial_DIN0309_L9.0mm_D3.2mm_P12.70mm_Horizontal, symbol Device:R
- added R6, R7: 3k3, Resistor_THT:R_Axial_DIN0309_L9.0mm_D3.2mm_P12.70mm_Horizontal, symbol Device:R
- added R8, R9: 5k1, Resistor_THT:R_Axial_DIN0207_L6.3mm_D2.5mm_P7.62mm_Horizontal, symbol VGA_V11-cache:R
- added R?: 10, Resistor_THT:R_Axial_DIN0207_L6.3mm_D2.5mm_P7.62mm_Horizontal, symbol VGA_V11-cache:R
- added U1: 74LS240_Split, Package_DIP:DIP-20_W7.62mm_Socket, symbol 74xx:74LS240_Split
- added unit 3 of U15
- added unit 2 of U15
- added U16: CModA7, Package_DIP:DIP-48_W15.24mm_Socket, symbol MyLib:CModA7
- added U17: VDIP2-32, Package_DIP:DIP-32_W15.24mm_Socket, symbol MyLib:VDIP2-32
- added U19: LM741, Package_DIP:DIP-8_W7.62mm_Socket, symbol Amplifier_Operational:LM741
- added U20: LM386, Package_DIP:DIP-8_W7.62mm_Socket, symbol Amplifier_Audio:LM386
- RN3: renamed from RN?; footprint (none) -> Resistor_THT:R_Array_SIP9
- U14: renamed from U?; footprint (none) -> Package_DIP:DIP-16_W7.62mm_Socket
- U15, U2: renamed from U?; footprint (none) -> Package_DIP:DIP-14_W7.62mm_Socket
- gave numbers to parts that had none: 5
Connections:
- net +3.3V: now also R6.1, R7.1, U1.19, U1.20 (VCC), U15.10 (~{S}), U15.13 (~{R}), U15.14 (VCC); no longer X1.1 (EN), X1.14 (Vcc)
- net GCLK: now also U18.21 (CLK)
- net GND: now also C1.2, C14.2, C15.2, C32.2, C33.2, C36.2, J2.S, J3.S, R2.1, R3.1, R9.1, U1.1, U1.10 (GND), U1.11, U1.13, U1.15, U1.17, U15.11 (C), U15.12 (D), U15.7 (GND), U16.25 (GND), U17.18 (GND), U17.4 (GND), U17.5 (GND), U17.7 (GND), U20.2 (-), U20.4 (GND)
- net PH1: now also U15.5 (Q), U1.2; no longer U15.2 (D), U15.6 (~{Q})
- net PH2: now also U1.18, U16.27 (PIO27); no longer U15.5 (Q)
- net Q1: now also U16.39 (PIO39)
- net Q2: now also U16.38 (PIO38)
- net Q3: now also U16.37 (PIO37)
- net Q4: now also U16.36 (PIO36)
- net V7: now reaches R?.2, U18.17 (V7)
- net V7: now also U16.29 (PIO29)
- net V1: now reaches RN3.8 (R7), U18.11 (V1)
- net V1: now also U16.35 (PIO35)
- net V2: now reaches RN3.7 (R6), U18.12 (V2)
- net V2: now also U16.34 (PIO34)
- net V3: now reaches RN3.2 (R1), U18.13 (V3)
- net V3: now also U16.33 (PIO33)
- net V4: now reaches RN3.5 (R4), U18.14 (V4)
- net V4: now also U16.32 (PIO32)
- net V5: now reaches RN3.4 (R3), U18.15 (V5)
- net V5: now also U16.31 (PIO31)
- net V6: now reaches RN3.3 (R2), U18.16 (V6)
- net V6: now also U16.30 (PIO30)
- net V8: now reaches RN3.6 (R5), U18.18 (V8)
- net V8: now also U16.28 (PIO28)
- net at U18.22 (REF): now also U1.6
- net at U18.7 (X1/ICLK): now also U1.16; no longer X1.8 (OUT)
- new net: R8.1, R9.2, U20.3 (+)
- new net: C31.1, J2.T
- new net: C31.2, R3.2, U19.2 (-)
- new net: C34.1, U20.1 (GAIN)
- new net: C35.1, R?.2, U20.5
- new net: C34.2, U20.8 (GAIN)
- new net: C35.2, J3.T
- new net: U15.2 (D), U15.6 (~{Q})
- new net: U1.4, X1.8 (OUT)
- new net: R2.2, R4.1, U19.3 (+)
- new net: R4.2, R5.1, U19.6
- new net: C36.1, R?.1
- new net +12V: C33.1, U20.6 (V+)
- new net +5V: C1.1, C14.1, C15.1, U17.1 (+5V), U19.7 (V+), X1.1 (EN), X1.14 (Vcc)
- new net -5V: U19.4 (V-)
- new net ANAIN: R5.2, U16.15 (PIO15)
- new net AUD: C32.1, R8.2, U16.23 (PIO23)
- new net BA0: U16.48 (PIO48)
- new net BA1: U16.47 (PIO47)
- new net BA2: U16.46 (PIO46)
- new net BA3: U16.45 (PIO45)
- new net BA4: U16.44 (PIO44)
- new net BA5: U16.43 (PIO43)
- new net BA6: U16.42 (PIO42)
- new net BA7: U16.41 (PIO41)
- new net CTS0: U16.19 (PIO19), U17.9 (RTS)
- new net IRQ*: U16.12 (PIO12)
- new net OSC: U1.14
- new net RTS0: U16.20 (PIO20), U17.10 (CTS)
- new net RWB: U16.40 (PIO40)
- new net RxD0: U16.17 (PIO17), U17.6 (TxD)
- new net TxD0: U16.18 (PIO18), U17.8 (RxD)
- new net VDA: U16.14 (PIO14)
- new net VPA: U16.13 (PIO13)
- new net VPROG: R7.2, U16.22 (PIO22), U17.23 (PROG)
- new net VRESET: R6.2, U16.21 (PIO21), U17.22 (RESET)
- new net VU: U16.24 (VU)
- new net WA0: U16.1 (PIO1)
- new net WA1: U16.2 (PIO2)
- new net WA12: U16.8 (PIO8)
- new net WA13: U16.9 (PIO9)
- new net WA14: U16.10 (PIO10)
- new net WA15: U16.11 (PIO11)
- new net WA2: U16.3 (PIO3)
- new net WA3: U16.4 (PIO4)
- new net WA4: U16.5 (PIO5)
- new net WA5: U16.6 (PIO6)
- new net WA6: U16.7 (PIO7)
- no-connect marks 5 -> 15
Other:
- note added: "USB Host for keyboard / mouse"
- note removed: "Decode $D8xxxx"
- company: (none) -> Finitron
- title: (none) -> ISA65816 Clock Generator
- moved on the sheet: C18A, C18B, R?, RN2, RN3, U14, U15A, U18, U2A, U2B, X1

Commit message: ISA65816 - update
Parts:
- C1, C14, C15, C31: footprint (none) -> Capacitor_THT:C_Disc_D3.8mm_W2.6mm_P2.50mm
- C18A1: renamed from C18A; footprint (none) -> Capacitor_THT:C_Disc_D3.8mm_W2.6mm_P2.50mm
- C18B1: renamed from C18B; footprint (none) -> Capacitor_THT:C_Disc_D3.8mm_W2.6mm_P2.50mm
- R10: renamed from R?; footprint Resistor_THT:R_Axial_DIN0207_L6.3mm_D2.5mm_P7.62mm_Horizontal -> Resistor_THT:R_Axial_DIN0204_L3.6mm_D1.6mm_P5.08mm_Horizontal
- R12: renamed from R?; footprint (none) -> Resistor_THT:R_Axial_DIN0204_L3.6mm_D1.6mm_P5.08mm_Horizontal
- R2, R3, R4, R5, R6, R7: footprint Resistor_THT:R_Axial_DIN0309_L9.0mm_D3.2mm_P12.70mm_Horizontal -> Resistor_THT:R_Axial_DIN0204_L3.6mm_D1.6mm_P5.08mm_Horizontal
- R8, R9: footprint Resistor_THT:R_Axial_DIN0207_L6.3mm_D2.5mm_P7.62mm_Horizontal -> Resistor_THT:R_Axial_DIN0204_L3.6mm_D1.6mm_P5.08mm_Horizontal
Connections:
- net VPA is gone; now on net WA12: U16.13 (PIO13)
- net +3.3V: now also C1.1, C14.1, C15.1, RN2.1 (common); no longer U18.19 (~{PD}), U18.25 (R1), U18.26 (R2), U18.27 (R3), U18.4 (S1)
- net +5V: no longer C1.1, C14.1, C15.1
- net WA12: no longer U16.8 (PIO8)
- net IRQ1*: now reaches U16.26 (PIO26)
- net IRQ* renamed WA11
- net WA13 renamed WA8
- net WA14 renamed WA9
- net WA15 renamed WA10
- new net WA7: U16.8 (PIO8)
- no-connect marks 15 -> 29
Other:
- moved on the sheet: R9
