File: ISA/ISA65816/ISA65816.kicad_sch (KiCad schematic)
At the start: 23 parts, among them J1 Bus_ISA_16bit, U3 74LVC245, U4 74LVC245, U5 W65C816SP, U6 74LVC245, U7 74LVC573, U8 74LVC245

Commit message: ISA65816 - update
Parts:
- removed U?: 74LVC08, symbol 74xx:74LS08
- removed U?: 74LVC04, symbol 74xx:74LS04
- added C10, C11, C3, C4, C6, C7, C8, C9: 0.1u, symbol Device:C
- added U1: 74LS240_Split, Package_DIP:DIP-20_W7.62mm_Socket, symbol 74xx:74LS240_Split
- added U2: 74LVC00, Package_DIP:DIP-14_W7.62mm_Socket, symbol 74xx:74LS00
- D1: renamed from D?; footprint (none) -> Diode_THT:D_A-405_P10.16mm_Horizontal
- J1: footprint (none) -> Connector_PCBEdge:BUS_AT
- R1: footprint (none) -> Resistor_THT:R_Axial_DIN0204_L3.6mm_D1.6mm_P7.62mm_Horizontal
- U10, U9: renamed from U?; footprint (none) -> Package_DIP:DIP-20_W7.62mm_Socket
- U11: renamed from U5; footprint (none) -> Package_DIP:DIP-40_W15.24mm_Socket
- U12, U13: renamed from U?; footprint (none) -> Package_DIP:DIP-48_W15.24mm_Socket
- U21, U22: renamed from U?; footprint (none) -> Package_TO_SOT_THT:TO-92
- gave numbers to parts that had none: 3
Connections:
- net +5V: now also C10.1, C11.1, C3.1, C4.1, C6.1, C7.1, C8.1, C9.1
- net ABORTB: now also U11.3 (ABORTB)
- net BE: now also RN1.2 (R1), U2.9
- net GND: now also C10.2, C11.2, C3.2, C4.2, C6.2, C7.2, C8.2, C9.2
- net IRQ*: now also RN1.5 (R4)
- net PH2: now also U2.10; no longer U11.37 (PH2-IN)
- net RESB: now also U1.8
- net RESET: now also U1.12
- new net: U11.37 (PH2-IN), U2.11
- new net: U2.12, U2.13, U2.8
- no-connect marks 15 -> 17
Other:
- removed sheet IRQ
- removed sheet IRQFPGA
- company: (none) -> Finitron
- title: (none) -> ISA65816 CPU Card

Commit message: ISA65816 - update
Parts:
- added C50, C51: 10u, Capacitor_THT:CP_Radial_D5.0mm_P2.50mm, symbol Device:C
- added R11: 10k, Resistor_THT:R_Axial_DIN0204_L3.6mm_D1.6mm_P5.08mm_Horizontal, symbol Device:R
- added RN4: 10k, Resistor_THT:R_Array_SIP9, symbol Device:R_Network08
- added unit 5 of U2
- added U50: AMS1117-3.3, Package_TO_SOT_SMD:SOT-223-3_TabPin2, symbol Regulator_Linear:AMS1117-3.3
- C10, C11, C3, C4, C6, C7, C8, C9: footprint (none) -> Capacitor_THT:C_Disc_D3.8mm_W2.6mm_P2.50mm
- C30: footprint (none) -> Capacitor_THT:CP_Radial_D5.0mm_P2.50mm
- JP1: footprint (none) -> Connector_PinHeader_2.54mm:PinHeader_1x02_P2.54mm_Vertical
- JP2: renamed from JP?; footprint (none) -> Connector_PinHeader_2.54mm:PinHeader_1x02_P2.54mm_Vertical
- R1: footprint (none) -> Resistor_THT:R_Axial_DIN0204_L3.6mm_D1.6mm_P5.08mm_Horizontal
- R52: renamed from R2; footprint (none) -> Resistor_THT:R_Axial_DIN0204_L3.6mm_D1.6mm_P5.08mm_Horizontal
- renumbered R1 to R51
Connections:
- net +3.3V: now also C10.1, C11.1, C3.1, C4.1, C6.1, C7.1, C8.1, C9.1, R51.1, C51.1, RN4.1 (common), U2.14 (VCC), U50.2 (VO)
- net +5V: now also J1.29 (VCC), J1.3 (+5V), J1.78 (+5V), C50.1, U50.3 (VI); no longer C10.1, C11.1, C3.1, C4.1, C6.1, C7.1, C8.1, C9.1
- net DACK0*: now also RN4.2 (R1)
- net DACK1*: now also RN4.3 (R2)
- net DACK2*: now also RN4.4 (R3)
- net DACK3*: now also RN4.5 (R4)
- net DACK5*: now also RN4.6 (R5)
- net DACK6*: now also RN4.7 (R6)
- net GND: now also C50.2, C51.2, R11.2, U2.7 (GND), U50.1 (GND); no longer J1.10 (GND), U6.11 (B7)
- net REFRESH*: now also RN4.8 (R7)
- net RESB: now also U11.40 (RESB)
- net TC: now also R11.1
- net -5V: now reaches J1.5 (-5V)
- net +12V: now reaches J1.9 (+12V)
- net DIRQ* renamed IRQ9*
- removed net VCC: J1.29 (VCC), J1.3 (+5V), J1.78 (+5V), R51.1
- no-connect marks 17 -> 32
Other:
- moved on the sheet: C10, C11, C3, C4, C6, C7, C8, C9, U2C, U2D
